Commit message: Add GIAR chest/back logo to all G1 URDF/MJCF variants
Scripted pipeline (trace_giar_wordmark.py + generate_logo_mesh.py +
apply_logo_to_models.py) traces the real GIAR wordmark from the brand
image and welds it as a cosmetic decal to torso_link on both front and
back, across all 10 G1 description variants.

Co-Authored-By: Claude Sonnet 5 <noreply@anthropic.com>
Claude-Session: https://claude.ai/code/session_01MtQdneuEj7mEdL3F1pxXd5

File: resources/robots/unitree_robotics/g1_description/g1_12dof.urdf (robot description, URDF)
Before this commit: robot g1_12dof, 31 links, 30 joints
Links:
- added link logo_back_link, mass 0.001; visual mesh filename=meshes/giar_logo_link.STL; visual mesh filename=meshes/giar_logo_link_accent.STL
- link logo_link: geometry visual mesh filename=meshes/giar_logo_link.STL; visual mesh filename=meshes/giar_logo_link_accent.STL
Joints:
- added joint logo_back_joint: type fixed, parent torso_link, child logo_back_link, origin xyz=-0.0686 0 0.2 rpy=0 0 3.14159265
- joint logo_joint: origin xyz=0.0039635 0 -0.044 rpy=0 0 0 -> xyz=0.0796 0 0.2 rpy=0 0 0

File: resources/robots/unitree_robotics/g1_description/g1_23dof.urdf (robot description, URDF)
Before this commit: robot g1_23dof, 33 links, 32 joints
Links:
- added link logo_back_link, mass 0.001; visual mesh filename=meshes/giar_logo_link.STL; visual mesh filename=meshes/giar_logo_link_accent.STL
- link logo_link: geometry visual mesh filename=meshes/giar_logo_link.STL; visual mesh filename=meshes/giar_logo_link_accent.STL
Joints:
- added joint logo_back_joint: type fixed, parent torso_link, child logo_back_link, origin xyz=-0.085 0 0.16 rpy=0 0 3.14159265
- joint logo_joint: origin xyz=0.0039635 0 -0.054 rpy=0 0 0 -> xyz=0.1 0 0.16 rpy=0 0 0

File: resources/robots/unitree_robotics/g1_description/g1_23dof_rev_1_0.urdf (robot description, URDF)
Before this commit: robot g1_23dof_rev_1_0, 31 links, 30 joints
Links:
- added link logo_back_link, mass 0.001; visual mesh filename=meshes/giar_logo_link.STL; visual mesh filename=meshes/giar_logo_link_accent.STL
- link logo_link: geometry visual mesh filename=meshes/giar_logo_link.STL; visual mesh filename=meshes/giar_logo_link_accent.STL
Joints:
- added joint logo_back_joint: type fixed, parent torso_link, child logo_back_link, origin xyz=-0.0686 0 0.2 rpy=0 0 3.14159265
- joint logo_joint: origin xyz=0.0039635 0 -0.044 rpy=0 0 0 -> xyz=0.0796 0 0.2 rpy=0 0 0

File: resources/robots/unitree_robotics/g1_description/g1_29dof.urdf (robot description, URDF)
Before this commit: robot g1_29dof, 40 links, 39 joints
Links:
- added link logo_back_link, mass 0.001; visual mesh filename=meshes/giar_logo_link.STL; visual mesh filename=meshes/giar_logo_link_accent.STL
- link logo_link: geometry visual mesh filename=meshes/giar_logo_link.STL; visual mesh filename=meshes/giar_logo_link_accent.STL
Joints:
- added joint logo_back_joint: type fixed, parent torso_link, child logo_back_link, origin xyz=-0.085 0 0.16 rpy=0 0 3.14159265
- joint logo_joint: origin xyz=0.0039635 0 -0.054 rpy=0 0 0 -> xyz=0.1 0 0.16 rpy=0 0 0

File: resources/robots/unitree_robotics/g1_description/g1_29dof_lock_waist.urdf (robot description, URDF)
Before this commit: robot g1_29dof_lock_waist, 40 links, 39 joints
Links:
- added link logo_back_link, mass 0.001; visual mesh filename=meshes/giar_logo_link.STL; visual mesh filename=meshes/giar_logo_link_accent.STL
- link logo_link: geometry visual mesh filename=meshes/giar_logo_link.STL; visual mesh filename=meshes/giar_logo_link_accent.STL
Joints:
- added joint logo_back_joint: type fixed, parent torso_link, child logo_back_link, origin xyz=-0.085 0 0.16 rpy=0 0 3.14159265
- joint logo_joint: origin xyz=0.0039635 0 -0.054 rpy=0 0 0 -> xyz=0.1 0 0.16 rpy=0 0 0

File: resources/robots/unitree_robotics/g1_description/g1_29dof_lock_waist_rev_1_0.urdf (robot description, URDF)
Before this commit: robot g1_29dof_lock_waist_rev_1_0, 39 links, 38 joints
Links:
- added link logo_back_link, mass 0.001; visual mesh filename=meshes/giar_logo_link.STL; visual mesh filename=meshes/giar_logo_link_accent.STL
- link logo_link: geometry visual mesh filename=meshes/giar_logo_link.STL; visual mesh filename=meshes/giar_logo_link_accent.STL
Joints:
- added joint logo_back_joint: type fixed, parent torso_link, child logo_back_link, origin xyz=-0.085 0 0.16 rpy=0 0 3.14159265
- joint logo_joint: origin xyz=0.0039635 0 -0.044 rpy=0 0 0 -> xyz=0.1 0 0.16 rpy=0 0 0

File: resources/robots/unitree_robotics/g1_description/g1_29dof_rev_1_0.urdf (robot description, URDF)
Before this commit: robot g1_29dof_rev_1_0, 39 links, 38 joints
Links:
- added link logo_back_link, mass 0.001; visual mesh filename=meshes/giar_logo_link.STL; visual mesh filename=meshes/giar_logo_link_accent.STL
- link logo_link: geometry visual mesh filename=meshes/giar_logo_link.STL; visual mesh filename=meshes/giar_logo_link_accent.STL
Joints:
- added joint logo_back_joint: type fixed, parent torso_link, child logo_back_link, origin xyz=-0.085 0 0.16 rpy=0 0 3.14159265
- joint logo_joint: origin xyz=0.0039635 0 -0.044 rpy=0 0 0 -> xyz=0.1 0 0.16 rpy=0 0 0

File: resources/robots/unitree_robotics/g1_description/g1_29dof_with_hand.urdf (robot description, URDF)
Before this commit: robot g1_29dof_with_hand, 54 links, 53 joints
Links:
- added link logo_back_link, mass 0.001; visual mesh filename=meshes/giar_logo_link.STL; visual mesh filename=meshes/giar_logo_link_accent.STL
- link logo_link: geometry visual mesh filename=meshes/giar_logo_link.STL; visual mesh filename=meshes/giar_logo_link_accent.STL
Joints:
- added joint logo_back_joint: type fixed, parent torso_link, child logo_back_link, origin xyz=-0.085 0 0.16 rpy=0 0 3.14159265
- joint logo_joint: origin xyz=0.0039635 0 -0.054 rpy=0 0 0 -> xyz=0.1 0 0.16 rpy=0 0 0

File: resources/robots/unitree_robotics/g1_description/g1_29dof_with_hand_rev_1_0.urdf (robot description, URDF)
Before this commit: robot g1_29dof_with_hand_rev_1_0, 53 links, 52 joints
Links:
- added link logo_back_link, mass 0.001; visual mesh filename=meshes/giar_logo_link.STL; visual mesh filename=meshes/giar_logo_link_accent.STL
- link logo_link: geometry visual mesh filename=meshes/giar_logo_link.STL; visual mesh filename=meshes/giar_logo_link_accent.STL
Joints:
- added joint logo_back_joint: type fixed, parent torso_link, child logo_back_link, origin xyz=-0.085 0 0.16 rpy=0 0 3.14159265
- joint logo_joint: origin xyz=0.0039635 0 -0.044 rpy=0 0 0 -> xyz=0.1 0 0.16 rpy=0 0 0

File: resources/robots/unitree_robotics/g1_description/g1_dual_arm.urdf (robot description, URDF)
Before this commit: robot g1_dual_arm, 26 links, 25 joints
Links:
- added link logo_back_link, mass 0.001; visual mesh filename=meshes/giar_logo_link.STL; visual mesh filename=meshes/giar_logo_link_accent.STL
- link logo_link: geometry visual mesh filename=meshes/giar_logo_link.STL; visual mesh filename=meshes/giar_logo_link_accent.STL
Joints:
- added joint logo_back_joint: type fixed, parent torso_link, child logo_back_link, origin xyz=-0.085 0 0.16 rpy=0 0 3.14159265
- joint logo_joint: origin xyz=0.0039635 0 -0.054 rpy=0 0 0 -> xyz=0.1 0 0.16 rpy=0 0 0
